File: seedsigner-esp32-dev-board.kicad_pcb (KiCad board)
At the start: 2 copper layers, 70 x 78 mm, 14 parts, among them J1 Conn_01x06, J2 Conn_01x04, U1 ESP32-S2-SAOLA-1M, U2 OV_CAMERA, U3 RASPBERRY_PI_3_MODEL_B+

Commit message: final gerbers and zip
Routing:
- net /BACKLIGHT: track 14.5 -> 12.5 mm
Other:
- board text added: "BACKLIGHT SELECT"
- board text added: "MAX"
- board text added: "PWM"
Changed lines of the file:
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@@
       (drillshape 0)
       (scaleselection 1)
-      (outputdirectory "gerbers/take2/")
+      (outputdirectory "gerbers/take3/")
     )
   )
@@
     (property "Sheetname" "")
     (attr exclude_from_pos_files)
-    (fp_text reference "JP1" (at 4.079 0.127) (layer "B.SilkS")
+    (fp_text reference "JP1" (at -3.175 0) (layer "B.SilkS")
       (effects (font (size 1 1) (thickness 0.15)) (justify mirror))
     )
@@
     (property "Sheetname" "")
     (attr exclude_from_pos_files)
-    (fp_text reference "JP2" (at 3.175 0) (layer "B.SilkS")
+    (fp_text reference "JP2" (at -3.175 0) (layer "B.SilkS")
       (effects (font (size 1 1) (thickness 0.15)) (justify mirror))
     )
@@
     (effects (font (size 0.7 0.7) (thickness 0.125)) (justify mirror))
   )
+  (gr_text "MAX" (at 37.973 -14.097) (layer "B.SilkS")
+    (effects (font (size 1 1) (thickness 0.25)) (justify mirror))
+  )
   (gr_text "3.3V" (at 14.224 -72.898 270) (layer "B.SilkS")
     (effects (font (size 0.7 0.7) (thickness 0.125)) (justify mirror))
@@
     (effects (font (size 0.7 0.7) (thickness 0.125)) (justify mirror))
   )
+  (gr_text "BACKLIGHT\nSELECT" (at 41.021 -19.812) (layer "B.SilkS")
+    (effects (font (size 1 1) (thickness 0.25)) (justify mirror))
+  )
+  (gr_text "PWM" (at 37.846 -16.764) (layer "B.SilkS")
+    (effects (font (size 1 1) (thickness 0.25)) (justify mirror))
+  )
   (gr_text "TX" (at 19.304 -73.406 270) (layer "B.SilkS")
     (effects (font (size 0.7 0.7) (thickness 0.125)) (justify mirror))
@@
   (segment (start 28.702 -59.944) (end 58.928 -59.944) (width 0.25) (layer "B.Cu") (net 56))
   (segment (start 58.928 -59.944) (end 60.96 -61.976) (width 0.25) (layer "B.Cu") (net 56))
-  (segment (start 43.688 -12.446) (end 43.688 -13.843) (width 0.25) (layer "F.Cu") (net 58))
-  (segment (start 40.767 -9.525) (end 43.688 -12.446) (width 0.25) (layer "F.Cu") (net 58))
-  (segment (start 39.48 -5.54) (end 40.767 -6.827) (width 0.25) (layer "F.Cu") (net 58))
-  (segment (start 40.767 -6.827) (end 40.767 -9.525) (width 0.25) (layer "F.Cu") (net 58))
-  (via (at 43.688 -13.843) (size 0.8) (drill 0.4) (layers "F.Cu" "B.Cu") (net 58))
+  (segment (start 40.767 -6.827) (end 39.48 -5.54) (width 0.25) (layer "F.Cu") (net 58))
+  (segment (start 40.767 -11.049) (end 40.767 -6.827) (width 0.25) (layer "F.Cu") (net 58))
+  (segment (start 42.037 -12.319) (end 40.767 -11.049) (width 0.25) (layer "F.Cu") (net 58))
+  (via (at 42.037 -12.319) (size 0.8) (drill 0.4) (layers "F.Cu" "B.Cu") (net 58))
+  (segment (start 42.052 -12.334) (end 42.037 -12.319) (width 0.25) (layer "B.Cu") (net 58))
   (segment (start 42.067 -13.843) (end 42.067 -16.622) (width 0.25) (layer "B.Cu") (net 58))
-  (segment (start 43.688 -13.843) (end 42.067 -13.843) (width 0.25) (layer "B.Cu") (net 58))
   (segment (start 42.067 -16.622) (end 42.052 -16.637) (width 0.25) (layer "B.Cu") (net 58))
+  (segment (start 42.052 -14.224) (end 42.052 -12.334) (width 0.25) (layer "B.Cu") (net 58))
   (segment (start 11.684 -75.692) (end 11.684 -72.644) (width 0.25) (layer "F.Cu") (net 59))
   (segment (start 17.78 -66.548) (end 17.78 -63.5) (width 0.25) (layer "F.Cu") (net 59))
